Commit message: breakpoint 1

File: urdf/robot1_base_01_cam.urdf (robot description, URDF)
Before this commit: robot robot1_xacro, 7 links, 6 joints
Links:
- added link rplidar_link, mass 1e-5; collision mesh filename=package://slam_car/meshes/rplidar2.STL; visual mesh filename=package://slam_car/meshes/rplidar2.STL
Joints:
- added joint rplidar_joint: type fixed, parent base_link, child rplidar_link, origin xyz=-0.125 0 0.11 rpy=0 0 0

File: urdf/robot1_base_01_cam.xacro (robot description, xacro)
@@ -174,5 +174,5 @@
   </link>
   <joint name="rplidar_joint" type="fixed">
-	<origin xyz="-0.125 0 0.125" rpy="0 0 0"/>
+	<origin xyz="-0.125 0 0.11" rpy="0 0 0"/>
 	<parent link="base_link"/>
 	<child link="rplidar_link"/>
@@ -196,5 +196,5 @@
     </visual>
     <inertial>
-      <mass value="0.2839" />
+      <mass value="1e-5" />
       <origin xyz="0 0 0" rpy="0 0 0" />
 	  <inertia ixx="1e-6" ixy="0" ixz="0" iyy="1e-6" iyz="0" izz="1e-6" />
